File: Battery/Battery.sch (KiCad schematic (older format))
At the start: 1 part

Commit message: Battery project netlist
Parts:
- BT1: footprint (none) -> Battery_Holder:SMTU2032-LF
Changed lines of the file:
@@
 F 0 "BT1" H 3768 3046 50  0000 L CNN
 F 1 "Coin_Battery_Cell" H 3768 2955 50  0000 L CNN
-F 2 "" V 3650 3010 50  0001 C CNN
+F 2 "Battery_Holder:SMTU2032-LF" V 3650 3010 50  0001 C CNN
 F 3 "~" V 3650 3010 50  0001 C CNN
 	1    3650 2950

Commit message: Battery Footprints 1.1
Parts:
- BT1: footprint Battery_Holder:SMTU2032-LF -> Battery_Holder:NH5077-LF
Changed lines of the file:
@@
 F 0 "BT1" H 3768 3046 50  0000 L CNN
 F 1 "Coin_Battery_Cell" H 3768 2955 50  0000 L CNN
-F 2 "Battery_Holder:SMTU2032-LF" V 3650 3010 50  0001 C CNN
+F 2 "Battery_Holder:NH5077-LF" V 3650 3010 50  0001 C CNN
 F 3 "~" V 3650 3010 50  0001 C CNN
 	1    3650 2950
@@
 $EndComp
 $Comp
-L power:+3V3 #PWR?
+L power:+3V3 #PWR0101
 U 1 1 5FB77249
 P 3650 2650
-F 0 "#PWR?" H 3650 2500 50  0001 C CNN
+F 0 "#PWR0101" H 3650 2500 50  0001 C CNN
 F 1 "+3V3" H 3665 2823 50  0000 C CNN
 F 2 "" H 3650 2650 50  0001 C CNN
@@
 $EndComp
 $Comp
-L power:GND #PWR?
+L power:GND #PWR0102
 U 1 1 5FB77282
 P 3650 3150
-F 0 "#PWR?" H 3650 2900 50  0001 C CNN
+F 0 "#PWR0102" H 3650 2900 50  0001 C CNN
 F 1 "GND" H 3655 2977 50  0000 C CNN
 F 2 "" H 3650 3150 50  0001 C CNN
