File: Single_transistor_AMP/Single_transistor_AMP.kicad_pcb (KiCad board)
At the start: 2 copper layers, 0 parts

Commit message: Single_Transistor_AMP PCB Layout created
Parts:
- added C1: 20uF, Capacitors_SMD:C_1206_HandSoldering, F.Cu at (99.1, 62.2)
- added C2: 47uF, Capacitors_SMD:C_1206_HandSoldering, F.Cu at (102.9, 69.8)
- added C3: 20uF, Capacitors_SMD:C_1206_HandSoldering, F.Cu at (109.2, 62.2)
- added C4: 20uF, Capacitors_SMD:C_1206_HandSoldering, F.Cu at (120.7, 62.2)
- added C5: 47uF, Capacitors_SMD:C_1206_HandSoldering, F.Cu at (115.6, 69.8)
- added J1: Power_Supply, Terminal_Blocks:TerminalBlock_bornier-2_P5.08mm, F.Cu at (111.8, 53.3)
- added J2: Signal_In, Terminal_Blocks:TerminalBlock_bornier-2_P5.08mm, F.Cu at (92.7, 59.7)
- added J3: Signal_Out, Terminal_Blocks:TerminalBlock_bornier-2_P5.08mm, F.Cu at (127.0, 64.8)
- added Q1: BC548, TO_SOT_Packages_THT:TO-92_Inline_Narrow_Oval, F.Cu at (102.9, 61.0)
- added Q2: BC548, TO_SOT_Packages_THT:TO-92_Inline_Narrow_Oval, F.Cu at (115.6, 61.0)
- added R1: 24k, Resistors_SMD:R_1206_HandSoldering, F.Cu at (99.1, 54.6)
- added R2: 6k8, Resistors_SMD:R_1206_HandSoldering, F.Cu at (100.3, 69.8)
- added R3: 4k7, Resistors_SMD:R_1206_HandSoldering, F.Cu at (101.6, 54.6)
- added R4: 1k8, Resistors_SMD:R_1206_HandSoldering, F.Cu at (105.4, 69.8)
- added R5: 24k, Resistors_SMD:R_1206_HandSoldering, F.Cu at (116.8, 54.6)
- added R6: 6k8, Resistors_SMD:R_1206_HandSoldering, F.Cu at (113.0, 69.8)
- added R7: 4k7, Resistors_SMD:R_1206_HandSoldering, F.Cu at (119.4, 54.6)
- added R8: 1k8, Resistors_SMD:R_1206_HandSoldering, F.Cu at (118.1, 69.8)
Other:
- board outline added: 47 x 28 mm

Commit message: Single_Transistor_AMP PCB routing
Routing:
- net /VCC: track 0.00 -> 22.1 mm
- net Net-(C3-Pad1): track 0.00 -> 20.0 mm
- net Net-(C1-Pad1): track 0.00 -> 15.3 mm
- net Net-(C3-Pad2): track 0.00 -> 9.75 mm
- net Net-(C4-Pad2): track 0.00 -> 9.53 mm
- net Net-(C5-Pad2): track 0.00 -> 6.89 mm
- net Net-(C2-Pad2): track 0.00 -> 6.89 mm
- net Net-(C1-Pad2): track 0.00 -> 6.57 mm
- net Net-(C4-Pad1): track 0.00 -> 6.57 mm
- added copper zone on B.Cu, net /GND
- added copper zone on F.Cu, net /GND
Changed lines of the file:
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@@
     (thickness 1.6)
     (drawings 18)
-    (tracks 0)
+    (tracks 48)
     (zones 0)
     (modules 18)
@@
     (aux_axis_origin 0 0)
     (grid_origin 109.22 62.23)
-    (visible_elements FFFFFF7F)
+    (visible_elements 7FFFFFFF)
     (pcbplotparams
       (layerselection 0x010fc_ffffffff)
@@
     (uvia_dia 0.3)
     (uvia_drill 0.1)
-    (add_net /GND)
-    (add_net /VCC)
     (add_net "Net-(C1-Pad1)")
     (add_net "Net-(C1-Pad2)")
@@
     (uvia_dia 0.3)
     (uvia_drill 0.1)
+    (add_net /GND)
+    (add_net /VCC)
   )
   (module Capacitors_SMD:C_1206_HandSoldering (layer F.Cu)
@@
   (gr_line (start 132.22 54.23) (end 132.22 68.23) (layer Margin) (width 1))
   (gr_line (start 93.22 48.23) (end 126.22 48.23) (layer Margin) (width 1))
+  (segment (start 98.52 59.69) (end 99.06 60.23) (width 0.5) (layer F.Cu) (net 1))
+  (segment (start 92.71 59.69) (end 98.52 59.69) (width 0.5) (layer F.Cu) (net 1))
+  (segment (start 99.06 56.76) (end 100.72 58.42) (width 0.5) (layer F.Cu) (net 2))
+  (segment (start 99.06 56.61) (end 99.06 56.76) (width 0.5) (layer F.Cu) (net 2))
+  (segment (start 102.87 62.23) (end 100.72 62.23) (width 0.5) (layer F.Cu) (net 2))
+  (segment (start 100.72 58.42) (end 100.72 62.23) (width 0.5) (layer F.Cu) (net 2))
+  (segment (start 99.06 64.03) (end 99.06 64.23) (width 0.5) (layer F.Cu) (net 2))
+  (segment (start 100.72 62.23) (end 100.72 62.37) (width 0.5) (layer F.Cu) (net 2))
+  (segment (start 100.72 62.37) (end 99.06 64.03) (width 0.5) (layer F.Cu) (net 2))
+  (segment (start 99.06 66.58) (end 100.33 67.85) (width 0.5) (layer F.Cu) (net 2))
+  (segment (start 99.06 64.23) (end 99.06 66.58) (width 0.5) (layer F.Cu) (net 2))
+  (segment (start 102.87 67.85) (end 102.87 63.5) (width 0.5) (layer F.Cu) (net 3))
+  (segment (start 102.87 67.85) (end 105.41 67.85) (width 0.5) (layer F.Cu) (net 3))
+  (segment (start 102.87 57.88) (end 102.87 60.96) (width 0.5) (layer F.Cu) (net 4))
+  (segment (start 101.6 56.61) (end 102.87 57.88) (width 0.5) (layer F.Cu) (net 4))
+  (segment (start 105.95 60.96) (end 107.22 62.23) (width 0.5) (layer F.Cu) (net 4))
+  (segment (start 102.87 60.96) (end 105.95 60.96) (width 0.5) (layer F.Cu) (net 4))
+  (segment (start 116.84 56.76) (end 113.22 60.38) (width 0.5) (layer F.Cu) (net 5))
+  (segment (start 116.84 56.61) (end 116.84 56.76) (width 0.5) (layer F.Cu) (net 5))
+  (segment (start 113.22 61.73) (end 113.72 62.23) (width 0.5) (layer F.Cu) (net 5))
+  (segment (start 113.72 62.23) (end 113.22 62.23) (width 0.5) (layer F.Cu) (net 5))
+  (segment (start 115.57 62.23) (end 113.72 62.23) (width 0.5) (layer F.Cu) (net 5))
+  (segment (start 113.22 61.73) (end 113.22 62.23) (width 0.5) (layer F.Cu) (net 5))
+  (segment (start 113.22 60.38) (end 113.22 61.73) (width 0.5) (layer F.Cu) (net 5))
+  (segment (start 113.22 61.73) (end 112.72 62.23) (width 0.5) (layer F.Cu) (net 5))
+  (segment (start 113.22 62.23) (end 112.72 62.23) (width 0.5) (layer F.Cu) (net 5))
+  (segment (start 112.72 62.23) (end 111.22 62.23) (width 0.5) (layer F.Cu) (net 5))
+  (segment (start 112.72 62.23) (end 113.22 62.73) (width 0.5) (layer F.Cu) (net 5))
+  (segment (start 113.22 62.73) (end 113.22 62.23) (width 0.5) (layer F.Cu) (net 5))
+  (segment (start 113.72 62.23) (end 113.22 62.73) (width 0.5) (layer F.Cu) (net 5))
+  (segment (start 113.22 67.66) (end 113.03 67.85) (width 0.5) (layer F.Cu) (net 5))
+  (segment (start 113.22 62.73) (end 113.22 67.66) (width 0.5) (layer F.Cu) (net 5))
+  (segment (start 116.3 60.23) (end 115.57 60.96) (width 0.5) (layer F.Cu) (net 6))
+  (segment (start 120.65 60.23) (end 116.3 60.23) (width 0.5) (layer F.Cu) (net 6))
+  (segment (start 120.65 57.88) (end 120.65 60.23) (width 0.5) (layer F.Cu) (net 6))
+  (segment (start 119.38 56.61) (end 120.65 57.88) (width 0.5) (layer F.Cu) (net 6))
+  (segment (start 126.46 64.23) (end 127 64.77) (width 0.5) (layer F.Cu) (net 7))
+  (segment (start 120.65 64.23) (end 126.46 64.23) (width 0.5) (layer F.Cu) (net 7))
+  (segment (start 115.57 67.85) (end 118.11 67.85) (width 0.5) (layer F.Cu) (net 8))
+  (segment (start 115.57 63.5) (end 115.57 67.85) (width 0.5) (layer F.Cu) (net 8))
+  (segment (start 99.06 52.61) (end 101.6 52.61) (width 1) (layer F.Cu) (net 10))
+  (segment (start 109.559999 51.139999) (end 111.76 53.34) (width 1) (layer F.Cu) (net 10))
+  (segment (start 104.920001 51.139999) (end 109.559999 51.139999) (width 1) (layer F.Cu) (net 10))
+  (segment (start 103.45 52.61) (end 104.920001 51.139999) (width 1) (layer F.Cu) (net 10))
+  (segment (start 101.6 52.61) (end 103.45 52.61) (width 1) (layer F.Cu) (net 10))
+  (segment (start 116.11 53.34) (end 116.84 52.61) (width 1) (layer F.Cu) (net 10))
+  (segment (start 111.76 53.34) (end 116.11 53.34) (width 1) (layer F.Cu) (net 10))
+  (segment (start 116.84 52.61) (end 119.38 52.61) (width 1) (layer F.Cu) (net 10))
+  (zone (net 9) (net_name /GND) (layer F.Cu) (hatch edge 0.508)
+    (connect_pads (clearance 0.508))
+    (min_thickness 0.254)
+    (fill yes (arc_segments 16) (thermal_gap 0.508) (thermal_bridge_width 0.508))
+    (polygon
+      (pts
+        (xy 85.72 46.73) (xy 85.72 75.73) (xy 133.72 75.73) (xy 133.72 46.73)
+      )
+    )
+  )
+  (zone (net 9) (net_name /GND) (layer B.Cu) (hatch edge 0.508)
+    (connect_pads (clearance 0.508))
+    (min_thickness 0.254)
+    (fill yes (arc_segments 16) (thermal_gap 0.508) (thermal_bridge_width 0.508))
+    (polygon
+      (pts
+        (xy 85.72 46.73) (xy 85.72 75.73) (xy 133.72 75.73) (xy 133.72 46.73)
+      )
+    )
+  )
 )
